Commit message: update world, control

File: urdf/body.xacro (robot description, xacro)
@@ -17,15 +17,10 @@
       </inertial>
       <visual>
-        <!-- <origin xyz="${wheel_base/2} 0 ${vehicle_height/2}" rpy="0 0 0"/>
-        <geometry>
-          <box size="${vehicle_length} 0.9 ${vehicle_height}"/>
-        </geometry> -->
-        <!-- <origin xyz="${wheel_base/2} 0 ${vehicle_height/2}" rpy="0 ${-pi/2} ${pi/2}"/> -->
-        <origin xyz="0 0 0" rpy="0 0 0"/>
+       <origin xyz="0 0 0" rpy="0 0 0"/>
         <geometry>
           <mesh filename="package://self-driving-car/mesh/body.dae" scale="${wheel_base/2.85} 1 1"/>
         </geometry>
         <gazebo reference="${suffix}_link">
-  		<material>Gazebo/Black</material>
+  		<material value="Gazebo/Black"/>
 	</gazebo>
       </visual>

File: urdf/imu.xacro (robot description, xacro)
@@ -17,5 +17,5 @@
         <origin rpy="0 0 0" xyz="0 0 0"/>
         <gazebo reference="${suffix}_link">
-  		<material>Gazebo/Red</material>
+  		<material value="Gazebo/Red"/>
 	</gazebo>
       </visual>
@@ -27,10 +27,10 @@
                  izz="${(sensor_box*sensor_box+sensor_box*sensor_box)*mass/12.0}"/>
       </inertial>
-      <!-- <collision>
+      <collision>
         <origin rpy="0 0 0" xyz="0 0 0"/>
         <geometry>
           <box size="${sensor_box} ${sensor_box} ${sensor_box}"/>
         </geometry>
-      </collision> -->
+      </collision>
     </link>
     <!-- imu -->

File: urdf/monocular_camera.xacro (robot description, xacro)
@@ -17,5 +17,5 @@
         <origin rpy="0 0 0" xyz="0 0 0"/>
         <gazebo reference="${suffix}_link">
-  		<material>Gazebo/Red</material>
+  		<material value="Gazebo/Red"/>
 	</gazebo>
       </visual>
@@ -42,5 +42,5 @@
     <!-- camera -->
     <gazebo reference="${suffix}_link">
-      <material>Gazebo/Black</material>
+      <material value="Gazebo/Black"/>
       <sensor type="camera" name="${suffix}">
         <update_rate>${fps}</update_rate>

File: urdf/steering.xacro (robot description, xacro)
@@ -20,5 +20,5 @@
         <origin xyz="0 0 0" rpy="${pi/2} 0 0"/>
         <gazebo reference="${suffix}_link">
-  		<material>Gazebo/Black</material>
+  		<material value="Gazebo/Black"/>
 	</gazebo>
       </visual>
@@ -30,10 +30,10 @@
                  izz="${radius*radius*mass/4+length*length*mass/12}" />
       </inertial>
-      <!-- <collision>
+     <collision>
         <origin xyz="0 0 0" rpy="${pi/2} 0 0"/>
         <geometry>
           <cylinder radius="0.1" length="0.01" />
         </geometry>
-      </collision> -->
+      </collision>
     </link>
   </xacro:macro>
@@ -55,5 +55,5 @@
         <origin xyz="0 0 0" rpy="${pi/2} 0 0"/>
         <gazebo reference="${suffix}_link">
-  		<material>Gazebo/Black</material>
+  		<material value="Gazebo/Black"/>
 	</gazebo>
       </visual>

File: urdf/vehicle.xacro (robot description, xacro)
@@ -4,6 +4,4 @@
 	<xacro:include filename="$(find self-driving-car)/urdf/wheel.xacro" />
 	<xacro:include filename="$(find self-driving-car)/urdf/steering.xacro" />
-	<xacro:include filename="$(find velodyne_description)/urdf/HDL-32E.urdf.xacro"/>
-	<xacro:include filename="$(find velodyne_description)/urdf/VLP-16.urdf.xacro"/>
 	<xacro:include filename="$(find self-driving-car)/urdf/monocular_camera.xacro"/>
 	<xacro:include filename="$(find self-driving-car)/urdf/imu.xacro"/>
@@ -49,8 +47,4 @@
   <!-- ================ sensor ================ -->
 	<xacro:property name="calibration" value="${load_yaml('$(find self-driving-car)/config/calibration.yaml')}"/>
-  <HDL-32E parent="base_link" name="velodyne" topic="/points_raw" hz="10" samples="220" gpu="$(arg gpu)">
-    <origin xyz="${calibration['base_link2velodyne']['x']} ${calibration['base_link2velodyne']['y']} ${calibration['base_link2velodyne']['z']}"
-            rpy="${calibration['base_link2velodyne']['roll']} ${calibration['base_link2velodyne']['pitch']} ${calibration['base_link2velodyne']['yaw']}" />
-  </HDL-32E>
   <xacro:monocular_camera_macro suffix="camera" parent="base_link" namespace=""
                                 x="${calibration['base_link2camera']['x']}"

File: urdf/wheel.xacro (robot description, xacro)
@@ -20,5 +20,5 @@
         <origin xyz="0 0 0" rpy="0 0 ${yaw}"/>
         <gazebo reference="${suffix}_link">
-  		<material>Gazebo/Gray</material>
+  		<material value="Gazebo/Gray"/>
 	</gazebo>
       </visual>
@@ -26,5 +26,6 @@
         <origin xyz="0 0 0" rpy="0 0 0"/>
         <mass value="${mass}"/>
-        <inertia ixx="${mass*radius*radius/2}"  ixy="0"  ixz="0" iyy="${radius*radius*mass/4+width*width*mass/12}" iyz="0" izz="${radius*radius*mass/4+width*width*mass/12}" />
+        <inertia ixx="${mass*radius*radius/2}"  ixy="0"  ixz="0"
+        	iyy="${radius*radius*mass/4+width*width*mass/12}" iyz="0" izz="${radius*radius*mass/4+width*width*mass/12}" />
       </inertial>
       <collision>
